File: related-projects/rom-utilities/schematic/rom-utilities/rom-utilities.kicad_sch (KiCad schematic)
At the start: 1 part

Commit message: update to schematic
Parts:
- added U1: ~, symbol AT28C64B_Library:AT28C64B-15PC
Connections:
- net at A1.5V4 (5V): now also U1.28 (VCC)
- net D0: now reaches A1.D22
- net D0: now also U1.11 (D0)
- net D1: now reaches A1.D23
- net D1: now also U1.12 (D1)
- net D2: now reaches A1.D24
- net D2: now also U1.13 (D2)
- net D3: now reaches A1.D25
- net D3: now also U1.15 (D3)
- net D4: now reaches A1.D26
- net D4: now also U1.16 (D4)
- net D5: now reaches A1.D27
- net D5: now also U1.17 (D5)
- net D6: now reaches A1.D28
- net D6: now also U1.18 (D6)
- net D7: now reaches A1.D29
- net D7: now also U1.19 (D7)
- net A0: now reaches A1.D34
- net A0: now also U1.10 (A0)
- net A1: now reaches A1.D35
- net A1: now also U1.9 (A1)
- net A2: now reaches A1.D36
- net A2: now also U1.8 (A2)
- net A3: now reaches A1.D37
- net A3: now also U1.7 (A3)
- net A4: now reaches A1.D38
- net A4: now also U1.6 (A4)
- net A5: now reaches A1.D39
- net A5: now also U1.5 (A5)
- net A6: now reaches A1.D40
- net A6: now also U1.4 (A6)
- net A7: now reaches A1.D41
- net A7: now also U1.3 (A7)
- net A8: now reaches A1.D42
- net A8: now also U1.25 (A8)
- net A9: now reaches A1.D43
- net A9: now also U1.24 (A9)
- net A10: now reaches A1.D44
- net A10: now also U1.21 (A10)
- net A11: now reaches A1.D45
- net A11: now also U1.23 (A11)
- net A12: now reaches A1.D46
- net A12: now also U1.2 (A12)
- net at A1.D48: now also U1.27 (WE)
- net at A1.D50 (D50_MISO): now also U1.20 (CS)
- net at A1.D52 (D52_SCK): now also U1.22 (OE)
- net at A1.GND6 (GND): now also U1.14 (GND)
Other:
- title: (none) -> ROM Utilities Schematic
- moved on the sheet: A1
