File: jml-8-mini/schematic/address_decoding.kicad_sch (KiCad schematic)
At the start: 9 parts, among them J5 Address Decoding, U6 74LS04, U7 CD74HCT4514E, U8 74LS139, U9 74LS32

Commit message: change "JML-8 Mini" to "JML-8-Mini" in schematic description
Other:
- title: JML-8 Mini Schematic -> JML-8-Mini Schematic
Changed lines of the file:
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@@
   (paper "A4")
   (title_block
-    (title "JML-8 Mini Schematic")
+    (title "JML-8-Mini Schematic")
     (date "2023-10-02")
     (rev "A")
