File: jml-8-mini/schematic/jml-8-mini.kicad_pcb (KiCad board)
At the start: 4 copper layers, 99.9 x 99.9 mm, 48 parts, among them J1 BarrelJack, J2 SIO CHB, J3 UART, J5 Address Decoding, J6 Z80 Lines, SW1 Reset, SW2 Power, U1 Z80CPU, U10 74LS74, U11 NE555P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

Commit message: create REV C with new changes, update gerbers
Other:
- board text added: "Rev C"
- board text removed: "Rev B"
Changed lines of the file:
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@@
     (title "JML-8-Mini PCB")
     (date "2023-10-20")
-    (rev "B")
+    (rev "C")
   )
   (layers
@@
     (effects (font (size 1.016 1.016) (thickness 0.1524)) (justify left bottom mirror))
   )
-  (gr_text "Rev B" (at 194.183 59.69 90) (layer "F.SilkS")
+  (gr_text "Rev C" (at 194.183 59.69 90) (layer "F.SilkS")
     (effects (font (size 1.778 1.778) (thickness 0.22225)) (justify left bottom))
   )
