File: jml-8-mini/schematic/power_clock_reset.kicad_sch (KiCad schematic)
At the start: 21 parts, among them J1 BarrelJack, SW1 Reset, SW2 Power, U10 74LS74, U11 NE555P, U6 74LS04, X1 8MHz, X2 2.4576MHz

Commit message: change "JML-8 Mini" to "JML-8-Mini" in schematic description
Other:
- title: JML-8 Mini Schematic -> JML-8-Mini Schematic
Changed lines of the file:
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@@
   (paper "A4")
   (title_block
-    (title "JML-8 Mini Schematic")
+    (title "JML-8-Mini Schematic")
     (date "2023-10-02")
     (rev "A")

Commit message: fix two capacitor footprints being swapped
Parts:
- C2: footprint Capacitor_THT:C_Disc_D5.0mm_W2.5mm_P5.00mm -> Capacitor_THT:CP_Radial_D5.0mm_P2.50mm
- C3: footprint Capacitor_THT:CP_Radial_D5.0mm_P2.50mm -> Capacitor_THT:C_Disc_D5.0mm_W2.5mm_P5.00mm
Changed lines of the file:
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@@
       (effects (font (size 1.27 1.27)) (justify left))
     )
-    (property "Footprint" "Capacitor_THT:C_Disc_D5.0mm_W2.5mm_P5.00mm" (at 89.2302 65.405 0)
+    (property "Footprint" "Capacitor_THT:CP_Radial_D5.0mm_P2.50mm" (at 89.2302 65.405 0)
       (effects (font (size 1.27 1.27)) hide)
     )
@@
       (effects (font (size 1.27 1.27)) (justify left))
     )
-    (property "Footprint" "Capacitor_THT:CP_Radial_D5.0mm_P2.50mm" (at 42.2402 52.705 0)
-      (effects (font (size 1.27 1.27)) hide)
-    )
+    (property "Footprint" "Capacitor_THT:C_Disc_D5.0mm_W2.5mm_P5.00mm" (at 42.2402 52.705 0)
+      (effects (font (size 1.27 1.27)) hide)
+    )
