File: peripherals/jml-8-mini-vga/schematic/jml-8-mini-vga.kicad_pcb (KiCad board)
At the start: 2 copper layers, 68.7 x 74.4 mm, 15 parts, among them J1 VGA, J2 Z80, U1 Tang Nano 9K, U2 74LVC4245A, U3 74LVC4245A, X1 25.175MHz

Commit message: add address decoding circuitry, regenerate gerbers
Parts:
- added J3: Conn_01x02_Pin, Connector_PinHeader_2.54mm:PinHeader_1x02_P2.54mm_Vertical, F.Cu at (168.8, 112.1)
- added REF**: OSHW-Logo2_7.3x6mm_SilkScreen, Symbol:OSHW-Logo2_7.3x6mm_SilkScreen, F.Cu at (150.3, 110.6)
- moved U3 2.27 mm to (165.5, 104.5)
Connections:
- U1 pad 12: unconnected-(U1-34/IOB23B/RGB_VS-Pad12) -> /FPGA_D4
- U1 pad 13: unconnected-(U1-40/IOB33B/RGB_HS-Pad13) -> /FPGA_D3
- U1 pad 15: /FPGA_D4 -> /FPGA_D5
- U1 pad 16: /FPGA_D3 -> /FPGA_D6
- U1 pad 18: /FPGA_D5 -> /FPGA_D7
- U1 pad 19: /FPGA_D6 -> /FPGA_D1
- U1 pad 20: /FPGA_D7 -> /~{FPGA_Y0}
- U1 pad 21: /FPGA_D1 -> /~{FPGA_Q0}
- U3 pad 10: GND -> unconnected-(U3-A7-Pad10)
- U3 pad 18: unconnected-(U3-B3-Pad18) -> /~{FPGA_WR}
- U3 pad 19: unconnected-(U3-B2-Pad19) -> /~{FPGA_IORQ}
- U3 pad 20: /~{FPGA_WR} -> /~{FPGA_Y0}
- U3 pad 21: /~{FPGA_IORQ} -> /~{FPGA_Q0}
- U3 pad 3: /~{IORQ} -> /~{Q0}
- U3 pad 4: /~{WR} -> /~{Y0}
- U3 pad 5: GND -> /~{IORQ}
- U3 pad 6: GND -> /~{WR}
- U3 pad 7: GND -> unconnected-(U3-A4-Pad7)
- U3 pad 8: GND -> unconnected-(U3-A5-Pad8)
- U3 pad 9: GND -> unconnected-(U3-A6-Pad9)
Routing:
- net /~{FPGA_Y0}: track 0.00 -> 54.0 mm
- net /~{FPGA_Q0}: track 0.00 -> 53.2 mm
- net /~{Y0}: track 0.00 -> 8.21 mm
- net GND: track 14.4 -> 22.0 mm, vias 10 -> 8
- net /~{Q0}: track 0.00 -> 7.64 mm
- net +3.3V: track 80.0 -> 76.7 mm
- net /FPGA_D3: track 52.5 -> 55.7 mm
- net /FPGA_D4: track 53.3 -> 56.5 mm
- net /~{IORQ}: track 7.94 -> 10.5 mm
- net /FPGA_D5: track 51.7 -> 53.9 mm
- net /FPGA_D6: track 51.0 -> 53.1 mm
- net /~{FPGA_WR}: track 31.0 -> 29.5 mm
- net /~{FPGA_IORQ}: track 30.2 -> 28.7 mm
- net +5V: track 63.6 -> 62.2 mm
- net /FPGA_D7: track 50.5 -> 51.5 mm
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- removed copper zone on F.Cu, net GND
